Commit message: noetic simulation ok, bot not fixed in gazebo

File: rom2109_description/urdf/rom2109_short.urdf (robot description, URDF)
Before this commit: robot rom2109_description, 6 links, 5 joints
Links:
- link base_link: mass 2.3522 -> 2.3323; geometry collision mesh filename=package://rom2109_description/meshes/short/base_link.STL; visual mesh filename=package://rom2109_description/meshes/short/base_link.STL
- link camera: mass 0.0447522011433413 -> 0.044752; geometry collision mesh filename=package://rom2109_description/meshes/short/camera.STL; visual mesh filename=package://rom2109_description/meshes/short/camera.STL
- link left_wheel: mass 2.8826 -> 2.88257784807586; geometry collision mesh filename=package://rom2109_description/meshes/short/left_wheel.STL; visual mesh filename=package://rom2109_description/meshes/short/left_wheel.STL
- link lidar: mass 1.33076913637071 -> 1.3308; geometry collision mesh filename=package://rom2109_description/meshes/short/lidar.STL; visual mesh filename=package://rom2109_description/meshes/short/lidar.STL
- link plate1: mass 0 -> 0.376303345586596; geometry collision mesh filename=package://rom2109_description/meshes/short/plate1.STL; visual mesh filename=package://rom2109_description/meshes/short/plate1.STL
- link right_wheel: geometry collision mesh filename=package://rom2109_description/meshes/short/right_wheel.STL; visual mesh filename=package://rom2109_description/meshes/short/right_wheel.STL
Joints:
- joint camera_joint: origin xyz=0.1095 0.0055774 -0.0125 rpy=0 0 0 -> xyz=0.1095 0.00557736269756123 -0.0125000000000011 rpy=0 0 0
- joint left_wheel_joint: origin xyz=0 0.098333 0.02605 rpy=0 0 0 -> xyz=0 0.098332880094503 0.0260500000000002 rpy=0 0 0

File: rom2109_description/urdf/rom2109_short_gazebo.urdf (robot description, URDF)
Before this commit: robot rom2109_description, 6 links, 5 joints
Links:
- link base_link: mass 2.3522 -> 2.3323; geometry collision mesh filename=package://rom2109_description/meshes/short/base_link.STL; visual mesh filename=package://rom2109_description/meshes/short/base_link.STL
- link camera: mass 0.0447522011433413 -> 0.044752; geometry collision mesh filename=package://rom2109_description/meshes/short/camera.STL; visual mesh filename=package://rom2109_description/meshes/short/camera.STL
- link left_wheel: mass 2.8826 -> 2.88257784807586; geometry collision mesh filename=package://rom2109_description/meshes/short/left_wheel.STL; visual mesh filename=package://rom2109_description/meshes/short/left_wheel.STL
- link lidar: mass 1.33076913637071 -> 1.3308; geometry collision mesh filename=package://rom2109_description/meshes/short/lidar.STL; visual mesh filename=package://rom2109_description/meshes/short/lidar.STL
- link plate1: mass 0 -> 0.376303345586596; geometry collision mesh filename=package://rom2109_description/meshes/short/plate1.STL; visual mesh filename=package://rom2109_description/meshes/short/plate1.STL
- link right_wheel: geometry collision mesh filename=package://rom2109_description/meshes/short/right_wheel.STL; visual mesh filename=package://rom2109_description/meshes/short/right_wheel.STL
Joints:
- joint camera_joint: origin xyz=0.1095 0.0055774 -0.0125 rpy=0 0 0 -> xyz=0.1095 0.00557736269756123 -0.0125000000000011 rpy=0 0 0
- joint left_wheel_joint: origin xyz=0 0.098333 0.02605 rpy=0 0 0 -> xyz=0 0.098332880094503 0.0260500000000002 rpy=0 0 0

File: rom2109_description/urdf/rom2109_tall.urdf (robot description, URDF)
Before this commit: robot rom2109, 8 links, 7 joints
Links:
- link base_link: mass 2.41256345237752 -> 2.3926; geometry collision mesh filename=package://rom2109_description/meshes/tall/base_link.STL; visual mesh filename=package://rom2109_description/meshes/tall/base_link.STL
- link camera: mass 0.0447522001138537 -> 0.044752; geometry collision mesh filename=package://rom2109_description/meshes/tall/camera.STL; visual mesh filename=package://rom2109_description/meshes/tall/camera.STL
- link left_wheel: geometry collision mesh filename=package://rom2109_description/meshes/tall/left_wheel.STL; visual mesh filename=package://rom2109_description/meshes/tall/left_wheel.STL
- link lidar: geometry collision mesh filename=package://rom2109_description/meshes/tall/lidar.STL; visual mesh filename=package://rom2109_description/meshes/tall/lidar.STL
- link plate1: geometry collision mesh filename=package://rom2109_description/meshes/tall/plate1.STL; visual mesh filename=package://rom2109_description/meshes/tall/plate1.STL
- link plate2: mass 0.358814063727848 -> 0.35881; geometry collision mesh filename=package://rom2109_description/meshes/tall/plate2.STL; visual mesh filename=package://rom2109_description/meshes/tall/plate2.STL
- link plate3: mass 0.358814063727848 -> 0; geometry collision mesh filename=package://rom2109_description/meshes/tall/plate3.STL; visual mesh filename=package://rom2109_description/meshes/tall/plate3.STL
- link right_wheel: mass 2.88257784610314 -> 2.8826; geometry collision mesh filename=package://rom2109_description/meshes/tall/right_wheel.STL; visual mesh filename=package://rom2109_description/meshes/tall/right_wheel.STL
Joints:
- joint camera_joint: origin xyz=0.1095 0.00557736269756118 -0.0125000000000011 rpy=0 0 0 -> xyz=0.1095 0.0055774 -0.0125 rpy=0 0 0
- joint lidar_joint: origin xyz=0.0159981253913104 -0.00158018301594729 0.0325999999999999 rpy=0 0 0 -> xyz=0.015998 -0.0015802 0.0326 rpy=0 0 0

File: rom2109_description/urdf/rom2109_tall_gazebo.urdf (robot description, URDF)
Before this commit: robot rom2109, 8 links, 7 joints
Links:
- link base_link: mass 2.41256345237752 -> 2.3926; geometry collision mesh filename=package://rom2109_description/meshes/tall/base_link.STL; visual mesh filename=package://rom2109_description/meshes/tall/base_link.STL
- link camera: mass 0.0447522001138537 -> 0.044752; geometry collision mesh filename=package://rom2109_description/meshes/tall/camera.STL; visual mesh filename=package://rom2109_description/meshes/tall/camera.STL
- link left_wheel: geometry collision mesh filename=package://rom2109_description/meshes/tall/left_wheel.STL; visual mesh filename=package://rom2109_description/meshes/tall/left_wheel.STL
- link lidar: geometry collision mesh filename=package://rom2109_description/meshes/tall/lidar.STL; visual mesh filename=package://rom2109_description/meshes/tall/lidar.STL
- link plate1: geometry collision mesh filename=package://rom2109_description/meshes/tall/plate1.STL; visual mesh filename=package://rom2109_description/meshes/tall/plate1.STL
- link plate2: mass 0.358814063727848 -> 0.35881; geometry collision mesh filename=package://rom2109_description/meshes/tall/plate2.STL; visual mesh filename=package://rom2109_description/meshes/tall/plate2.STL
- link plate3: mass 0.358814063727848 -> 0; geometry collision mesh filename=package://rom2109_description/meshes/tall/plate3.STL; visual mesh filename=package://rom2109_description/meshes/tall/plate3.STL
- link right_wheel: mass 2.88257784610314 -> 2.8826; geometry collision mesh filename=package://rom2109_description/meshes/tall/right_wheel.STL; visual mesh filename=package://rom2109_description/meshes/tall/right_wheel.STL
Joints:
- joint camera_joint: origin xyz=0.1095 0.00557736269756118 -0.0125000000000011 rpy=0 0 0 -> xyz=0.1095 0.0055774 -0.0125 rpy=0 0 0
- joint lidar_joint: origin xyz=0.0159981253913104 -0.00158018301594729 0.0325999999999999 rpy=0 0 0 -> xyz=0.015998 -0.0015802 0.0326 rpy=0 0 0
