Commit message: add gazebo pkg

File: rom2109_description/urdf/rom2109_bot.urdf (robot description, URDF)
Before this commit: robot rom2109, 6 links, 5 joints
Links:
- removed link left_wheel_link
- removed link right_whel_link
- removed link rp_lidar_link
- removed link wifi_Link
- added link left_wheel, mass 2.8826; collision mesh filename=package://rom2109_description/meshes/bot/left_wheel.STL; visual mesh filename=package://rom2109_description/meshes/bot/left_wheel.STL
- added link right_wheel, mass 2.8826; collision mesh filename=package://rom2109_description/meshes/bot/right_wheel.STL; visual mesh filename=package://rom2109_description/meshes/bot/right_wheel.STL
- added link rp_lidar, mass 0.17402; collision mesh filename=package://rom2109_description/meshes/bot/rp_lidar.STL; visual mesh filename=package://rom2109_description/meshes/bot/rp_lidar.STL
- added link wifi, mass 0.46643; collision mesh filename=package://rom2109_description/meshes/bot/wifi.STL; visual mesh filename=package://rom2109_description/meshes/bot/wifi.STL
- link base_link: mass 2.0151 -> 2.8573
Joints:
- joint frame_joint: origin xyz=0.016132 3.6141E-05 -0.20083 rpy=0 0 0 -> xyz=0 0 0 rpy=0 0 0
- joint left_wheel_joint: axis 0 -1 0 -> 0 1 0; child left_wheel_link -> left_wheel; origin xyz=0.016132 0.098369 -0.17478 rpy=0 0 0 -> xyz=0 0.098333 0.02605 rpy=0 0 0
- joint right_wheel_joint: axis 0 -1 0 -> 0 1 0; child right_whel_link -> right_wheel; origin xyz=0.016132 3.6141E-05 -0.20083 rpy=0 0 0 -> xyz=0 -0.098333 0.02605 rpy=0 0 0
- joint rp_lidar_joint: child rp_lidar_link -> rp_lidar; origin xyz=0 0 0 rpy=0 0 0 -> xyz=-0.016132 -3.6141E-05 0.20083 rpy=0 0 0
- joint wifi_joint: child wifi_Link -> wifi; origin xyz=0.016132 3.6141E-05 -0.20083 rpy=0 0 0 -> xyz=0 0 0 rpy=0 0 0

File: rom2109_description/urdf/rom2109_bot_gazebo.urdf (robot description, URDF)
Before this commit: robot rom2109, 6 links, 5 joints
Links:
- removed link left_wheel_link
- removed link right_whel_link
- removed link rp_lidar_link
- removed link wifi_Link
- added link left_wheel, mass 2.8826; collision mesh filename=package://rom2109_description/meshes/bot/left_wheel.STL; visual mesh filename=package://rom2109_description/meshes/bot/left_wheel.STL
- added link right_wheel, mass 2.8826; collision mesh filename=package://rom2109_description/meshes/bot/right_wheel.STL; visual mesh filename=package://rom2109_description/meshes/bot/right_wheel.STL
- added link rp_lidar, mass 0.17402; collision mesh filename=package://rom2109_description/meshes/bot/rp_lidar.STL; visual mesh filename=package://rom2109_description/meshes/bot/rp_lidar.STL
- added link wifi, mass 0.46643; collision mesh filename=package://rom2109_description/meshes/bot/wifi.STL; visual mesh filename=package://rom2109_description/meshes/bot/wifi.STL
- link base_link: mass 2.0151 -> 2.8573
Joints:
- joint frame_joint: origin xyz=0.016132 3.6141E-05 -0.20083 rpy=0 0 0 -> xyz=0 0 0 rpy=0 0 0
- joint left_wheel_joint: axis 0 -1 0 -> 0 1 0; child left_wheel_link -> left_wheel; origin xyz=0.016132 0.098369 -0.17478 rpy=0 0 0 -> xyz=0 0.098333 0.02605 rpy=0 0 0
- joint right_wheel_joint: axis 0 -1 0 -> 0 1 0; child right_whel_link -> right_wheel; origin xyz=0.016132 3.6141E-05 -0.20083 rpy=0 0 0 -> xyz=0 -0.098333 0.02605 rpy=0 0 0
- joint rp_lidar_joint: child rp_lidar_link -> rp_lidar; origin xyz=0 0 0 rpy=0 0 0 -> xyz=-0.016132 -3.6141E-05 0.20083 rpy=0 0 0
- joint wifi_joint: child wifi_Link -> wifi; origin xyz=0.016132 3.6141E-05 -0.20083 rpy=0 0 0 -> xyz=0 0 0 rpy=0 0 0
