Commit message: gazebo sensor complete

File: rom2109_description/urdf/robot.urdf.xacro (robot description, xacro)
@@ -2,3 +2,7 @@
 <robot xmlns:xacro="http://www.ros.org/wiki/xacro"  name="rom2109">
     <xacro:include filename="rom2109_tall.xacro" />
+    <xacro:include filename="gazebo_control.xacro" />
+    <xacro:include filename="lidar.xacro" />
+    <xacro:include filename="camera.xacro" />
+    <!-- <xacro:include filename="camera3d.xacro" /> -->
 </robot>

File: rom2109_description/urdf/rom2109_tall.xacro (robot description, xacro)
@@ -412,3 +412,16 @@
       xyz="0 0 0" />
   </joint>
+  <!-- Colour -->
+  <gazebo reference="base_link">
+    <material>Gazebo/Black</material>
+  </gazebo>
+  <gazebo reference="plate1">
+    <material>Gazebo/Yellow</material>
+  </gazebo>
+   <gazebo reference="plate2">
+    <material>Gazebo/Yellow</material>
+  </gazebo>
+   <gazebo reference="plate3">
+    <material>Gazebo/Yellow</material>
+  </gazebo>
 </robot>
