Commit message: base_link to base_footprint

File: rom2109_description/urdf/gazebo_control.xacro (robot description, xacro)
@@ -13,5 +13,5 @@
             <!-- Output -->
             <odometry_frame>odom</odometry_frame>
-            <robot_base_frame>base_link</robot_base_frame>
+            <robot_base_frame>base_footprint</robot_base_frame>
             <publish_odom>true</publish_odom>
             <publish_odom_tf>true</publish_odom_tf>

File: rom2109_description/urdf/hw_ros2_control.xacro (robot description, xacro)
@@ -10,5 +10,5 @@
             <param name="baud_rate">57600</param>
             <param name="timeout">1000</param>
-            <param name="enc_counts_perrev">1320</param>
+            <param name="enc_counts_per_rev">1320</param>
         </hardware>
         <joint name="left_wheel_joint">

File: rom2109_description/urdf/robot_hw.urdf.xacro (robot description, xacro)
@@ -3,5 +3,5 @@
     <xacro:arg name="use_ros2_control" default="true"/>
     <xacro:arg name="use_depth_camera" default="false"/>
-    <xacro:include filename="rom2109_tall.xacro" />
+    <xacro:include filename="rom2109_core.xacro" />
     <xacro:include filename="lidar.xacro" />
     <xacro:include filename="hw_ros2_control.xacro" />

File: rom2109_description/urdf/robot_sim.urdf.xacro (robot description, xacro)
@@ -1,9 +1,9 @@
 <?xml version="1.0"?>
 <robot xmlns:xacro="http://www.ros.org/wiki/xacro"  name="rom2109">
-    <xacro:include filename="rom2109_tall.xacro" />
+    <xacro:include filename="rom2109_core.xacro" />
     <xacro:include filename="lidar.xacro" />
     <!-- <xacro:include filename="hw_ros2_control.xacro" />  -->
-    <!-- <xacro:include filename="ros2_control.xacro" />  -->
-    <xacro:include filename="gazebo_control.xacro" />
+    <xacro:include filename="ros2_control.xacro" />
+    <!-- <xacro:include filename="gazebo_control.xacro" /> -->
     <xacro:include filename="camera.xacro" />
     <!-- <xacro:include filename="camera3d.xacro" /> -->

File: rom2109_description/urdf/rom2109_core.xacro (robot description, xacro)
@@ -1,4 +1,10 @@
 <?xml version="1.0"?>
 <robot xmlns:xacro="http://www.ros.org/wiki/xacro">
+    <link name="base_footprint"></link>
+    <joint name="base_footprint_joint" type="fixed">
+      <parent link="base_footprint"/>
+      <child link="base_link"/>
+      <origin xyz="0 0 0" rpy="0 0 0"/>
+    </joint>
     <link
     name="base_link">

File: rom2109_description/urdf/ros2_control.xacro (robot description, xacro)
@@ -29,5 +29,5 @@
             <!-- Output -->
             <odometry_frame>odom</odometry_frame>
-            <robot_base_frame>base_link</robot_base_frame>
+            <robot_base_frame>base_footprint</robot_base_frame>
             <publish_odom>true</publish_odom>
             <publish_odom_tf>true</publish_odom_tf>
