Commit message: wheel_.cmd err

File: rom2109_description/urdf/hw_ros2_control.xacro (robot description, xacro)
@@ -1,32 +1,36 @@
 <?xml version="1.0"?>
 <robot xmlns:xacro="http://www.ros.org/wiki/xacro">
-    <ros2_control name="RealRobot" type="system">
+    <xacro:macro name="diffbot_ros2_control" params="name prefix">
+    <ros2_control name="${name}" type="system">
         <hardware>
+            <!-- <plugin>ros2_control_demo_example_2/DiffBotSystemHardware</plugin> -->
             <!-- <plugin>diffdrive_arduino/DiffDriveArduino</plugin> -->
-            <plugin>ros2_control_demo_example_2/DiffDriveStm32Hardware</plugin>
+            <plugin>diffdrive_stm32/DiffDriveStm32Hardware</plugin>
             <param name="left_wheel_name">left_wheel_joint</param>
             <param name="right_wheel_name">right_wheel_joint</param>
             <param name="loop_rate">30</param>
-            <param name="device">/home/mr_robot/robotController</param>
+            <!-- <param name="device">/home/mr_robot/robotController</param> -->
+            <param name="device">/dev/serial/by-id/usb-1a86_USB_Serial-if00-port0</param>
             <param name="baud_rate">115200</param>
-            <param name="timeout">1000</param>
-            <param name="enc_counts_per_rev">1320</param>
+            <param name="timeout_ms">1000</param>
+            <param name="enc_counts_per_rev">6533</param>
         </hardware>
         <joint name="left_wheel_joint">
-            <command_interface name="velocity">
-                <param name="min">-10</param>
-                <param name="max">10</param>
-            </command_interface>
+            <command_interface name="velocity"/>
+                <!-- <param name="min">-50</param>
+                <param name="max">50</param>
+            </command_interface> -->
+            <state_interface name="position"/>
             <state_interface name="velocity"/>
-            <state_interface name="position"/>
         </joint>
         <joint name="right_wheel_joint">
-            <command_interface name="velocity">
-                <param name="min">-10</param>
-                <param name="max">10</param>
-            </command_interface>
+            <command_interface name="velocity"/>
+                <!-- <param name="min">-50</param>
+                <param name="max">50</param>
+            </command_interface> -->
+            <state_interface name="position"/>
             <state_interface name="velocity"/>
-            <state_interface name="position"/>
         </joint>
     </ros2_control>
+    </xacro:macro>
 </robot>

File: rom2109_description/urdf/robot_hw_control.urdf.xacro (robot description, xacro)
@@ -1,6 +1,8 @@
 <?xml version="1.0"?>
 <robot xmlns:xacro="http://www.ros.org/wiki/xacro"  name="rom2109">
+    <xacro:arg name="prefix" default="" />
     <xacro:arg name="use_ros2_control" default="true"/>
     <xacro:include filename="rom2109_core.xacro" />
     <xacro:include filename="hw_ros2_control.xacro" />
+    <xacro:diffbot_ros2_control name="DiffBot" prefix="$(arg prefix)" />
 </robot>
